File: schematic/LED-Controller/LED-Controller.sch (KiCad schematic (older format))
At the start: 14 parts, among them J1 5V Power, J2 ICSP, J3 RCin, J4 Serial Connect, J5 TSW-102-08-L-T-RA, J6 TSW-102-08-L-T-RA, J7 TSW-102-08-L-T-RA, U1 PIC18F2xQ43-xSO

Commit message: Schematic text updated
Parts:
- D1: value LED -> LED-Red
Other:
- note added: "1-2 Power from 5V LED rail (default)\n2-3 Power from RC input"
Changed lines of the file:
@@
 P 6350 3750
 F 0 "D1" H 6343 3967 50  0000 C CNN
-F 1 "LED" H 6343 3876 50  0000 C CNN
+F 1 "LED-Red" H 6343 3876 50  0000 C CNN
 F 2 "LED_SMD:LED_0603_1608Metric_Pad1.05x0.95mm_HandSolder" H 6350 3750 50  0001 C CNN
 F 3 "~" H 6350 3750 50  0001 C CNN
@@
 P 8600 1850
 F 0 "J5" H 9000 2115 50  0000 C CNN
-F 1 "TSW-102-08-L-T-RA" H 9000 2024 50  0000 C CNN
+F 1 "TSW-102-08-L-T-RA" H 9000 2024 50  0001 C CNN
 F 2 "HDRRA6W64P254_3X2_508X254X810P" H 9250 1950 50  0001 L CNN
 F 3 "http://suddendocs.samtec.com/catalog_english/tsw_th.pdf" H 9250 1850 50  0001 L CNN
@@
 P 8600 3500
 F 0 "J6" H 9000 3765 50  0000 C CNN
-F 1 "TSW-102-08-L-T-RA" H 9000 3674 50  0000 C CNN
+F 1 "TSW-102-08-L-T-RA" H 9000 3674 50  0001 C CNN
 F 2 "HDRRA6W64P254_3X2_508X254X810P" H 9250 3600 50  0001 L CNN
 F 3 "http://suddendocs.samtec.com/catalog_english/tsw_th.pdf" H 9250 3500 50  0001 L CNN
@@
 P 8600 5350
 F 0 "J7" H 9000 5615 50  0000 C CNN
-F 1 "TSW-102-08-L-T-RA" H 9000 5524 50  0000 C CNN
+F 1 "TSW-102-08-L-T-RA" H 9000 5524 50  0001 C CNN
 F 2 "HDRRA6W64P254_3X2_508X254X810P" H 9250 5450 50  0001 L CNN
 F 3 "http://suddendocs.samtec.com/catalog_english/tsw_th.pdf" H 9250 5350 50  0001 L CNN
@@
 Text Notes 6950 4600 0    50   ~ 0
 GND
+Text Notes 3800 6250 0    50   ~ 0
+1-2 Power from 5V LED rail (default)\n2-3 Power from RC input
 $EndSCHEMATC
